Commit message: add robot description assignment

File: robot_description_norasheikhly/src/robot_description/urdf/robot.urdf.xacro (robot description, xacro)
@@ -16,7 +16,4 @@
   <xacro:property name="wheel_y_offset" value="0.225"/>
   <xacro:property name="wheel_z_offset" value="-0.05"/>
-  <!--caster wheel size -->
-  <xacro:property name="caster_wheel_radius" value="0.09"/>
-  <xacro:property name="caster_wheel_width" value="0.04"/>
   <!-- Base link -->
   <link name="base_link">
@@ -46,4 +43,5 @@
     </inertial>
   </link>
+<!-- Base footprint -->
   <link name="base_footprint"/>
   <joint name="base_footprint_joint" type="fixed">
@@ -53,5 +51,5 @@
   </joint>
   <!-- Define the wheel macro -->
-  <xacro:macro name="wheel" params="prefix x_reflect y_reflect wheel_radius wheel_width">
+  <xacro:macro name="wheel" params="prefix x_reflect y_reflect">
     <!-- Wheel link -->
     <link name="${prefix}_wheel_link">
@@ -83,4 +81,31 @@
       </inertial>
     </link>
+  <!-- Caster Wheel link -->
+    <link name="caster_wheel">
+      <visual>
+        <geometry>
+          <sphere radius= "0.04"/>
+        </geometry>
+        <material name="black">
+          <color rgba="0.1 0.1 0.1 1.0"/>
+        </material>
+      </visual>
+      <collision>
+        <geometry>
+          <sphere radius="0.04"/>
+        </geometry>
+      </collision>
+      <inertial>
+        <mass value="0.2"/>
+        <origin xyz="0 0 0"/>
+        <inertia
+          ixx="0.0001"
+          ixy="0.0"
+          ixz="0.0"
+          iyy="0.0001"
+          iyz="0.0"
+          izz="0.0001"/>
+      </inertial>
+    </link>
     <!-- Wheel joint -->
     <joint name="${prefix}_wheel_joint" type="continuous">
@@ -92,9 +117,16 @@
       <axis xyz="0 1 0"/>
     </joint>
-  </xacro:macro>
+    </xacro:macro>
+<!-- Caster joint -->
+    <joint name="caster_joint" type="fixed">
+      <parent link="base_link"/>
+      <child link="caster_wheel"/>
+      <origin
+        xyz="-0.15 0 -0.12"
+        rpy="0 0 0"/>
+    </joint>
   <!-- Instantiate wheels: front left, front right, and caster in the back -->
-  <xacro:wheel prefix="front_left"  x_reflect="1" y_reflect="1" wheel_radius="${wheel_radius}" wheel_width="${wheel_width}"/>
-  <xacro:wheel prefix="front_right" x_reflect="1" y_reflect="-1" wheel_radius="${wheel_radius}" wheel_width="${wheel_width}"/>
-  <xacro:wheel prefix="caster_wheel"   x_reflect="-1" y_reflect="0" wheel_radius="${caster_wheel_radius}" wheel_width="${caster_wheel_width}"/>
+  <xacro:wheel prefix="front_left"  x_reflect="1" y_reflect="1"/>
+  <xacro:wheel prefix="front_right" x_reflect="1" y_reflect="-1"/>
   <!-- LiDAR link -->
   <link name="lidar_link">

Commit message: Add complete robot simulation assignment

File: robot_description_norasheikhly/src/robot_description/urdf/robot.urdf.xacro (robot description, xacro)
@@ -4,4 +4,5 @@
   <xacro:property name="pi" value="3.141592653589793"/>
   <xacro:arg name="mesh_path" default="package://robot_description/meshes/"/>
+  <xacro:include filename="$(find robot_description)/urdf/robot.gazebo.xacro"/>
   <!-- Base properties -->
   <xacro:property name="base_length" value="0.6"/>
@@ -81,5 +82,15 @@
       </inertial>
     </link>
-  <!-- Caster Wheel link -->
+    <!-- Wheel joint -->
+    <joint name="${prefix}_wheel_joint" type="continuous">
+      <parent link="base_link"/>
+      <child link="${prefix}_wheel_link"/>
+      <origin
+        xyz="${x_reflect * wheel_x_offset} ${y_reflect * wheel_y_offset} ${wheel_z_offset}"
+        rpy="0 0 0"/>
+      <axis xyz="0 1 0"/>
+    </joint>
+    </xacro:macro>
+    <!-- Caster Wheel link -->
     <link name="caster_wheel">
       <visual>
@@ -108,14 +119,4 @@
       </inertial>
     </link>
-    <!-- Wheel joint -->
-    <joint name="${prefix}_wheel_joint" type="continuous">
-      <parent link="base_link"/>
-      <child link="${prefix}_wheel_link"/>
-      <origin
-        xyz="${x_reflect * wheel_x_offset} ${y_reflect * wheel_y_offset} ${wheel_z_offset}"
-        rpy="0 0 0"/>
-      <axis xyz="0 1 0"/>
-    </joint>
-    </xacro:macro>
 <!-- Caster joint -->
     <joint name="caster_joint" type="fixed">
@@ -126,4 +127,11 @@
         rpy="0 0 0"/>
     </joint>
+  <!-- Gazebo friction properties-Caster wheel -->
+  <gazebo reference = "caster_wheel">
+   <mu1>0.0</mu1>
+   <mu2>0.0</mu2>
+   <kp>1000000.0</kp>
+   <kd>100.0</kd>
+  </gazebo>
   <!-- Instantiate wheels: front left, front right, and caster in the back -->
   <xacro:wheel prefix="front_left"  x_reflect="1" y_reflect="1"/>
